File: schematics/src/mainboard/mainboard.brd (EAGLE design)
At the start: 81.3 x 99.1 mm, 105 parts, among them IC1 LM2904, IC2 LM2904, IC3 LM2904, T1 2SC945, T3 BC546B, T4 BC546B, T5 BC546B, T6 BC546B

Commit message: Some updates & bugfixes
Parts:
- moved BD1_CON 44.4 mm to (78.7, 81.3), turned to 90 degrees
- moved BD2_CON 44.4 mm to (34.3, 81.3)
Routing:
- net BD2_TUNE_A: track 55.5 -> 87.2 mm, vias 0 -> 2
- net BD1_TUNE_B: track 81.2 -> 105.1 mm, vias 0 -> 1
- net BD2_DECAY_B: track 51.0 -> 74.1 mm, vias 0 -> 3
- net BD1_TONE_A: track 73.4 -> 93.0 mm, vias 1 -> 2
- net BD1_TRIGGER: track 76.2 -> 86.4 mm
- net BD2_DECAY_A: track 37.3 -> 28.8 mm, vias 1 -> 0
- net BD2_TRIGGER: track 50.8 -> 42.5 mm
- net BD1_TUNE_A: track 77.8 -> 86.0 mm, vias 0 -> 2
- net N$23: track 44.3 -> 47.7 mm, vias 0 -> 1
Other:
- board text added: "TR82 mk2 Kicks v1.1 gerbster.nl 2022"
- board text removed: "TR82 mk2 Kicks v1.0 gerbster.nl 2021"

Commit message: Fixed orentation SD Decay pot
Parts:
- R18: value 6.6k -> 3.3k
Changed lines of the file:
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@@
 <attribute name="VALUE" x="45.974" y="54.102" size="1.27" layer="27" font="vector" ratio="11" rot="R180"/>
 </element>
-<element name="R18" library="rcl" library_urn="urn:adsk.eagle:library:334" package="0207/7" package3d_urn="urn:adsk.eagle:package:23493/2" value="6.6k" x="49.53" y="55.88" smashed="yes">
+<element name="R18" library="rcl" library_urn="urn:adsk.eagle:library:334" package="0207/7" package3d_urn="urn:adsk.eagle:package:23493/2" value="3.3k" x="49.53" y="55.88" smashed="yes">
 <attribute name="NAME" x="46.99" y="55.245" size="1.27" layer="25" font="vector" ratio="10"/>
 <attribute name="POPULARITY" value="22" x="49.53" y="55.88" size="1.778" layer="27" display="off"/>
