File: schematics/src/mainboard/mainboard.sch (EAGLE design)
At the start: 104 parts, among them IC1 LM2904, IC2 LM2904, IC3 LM2904, T1 2SC945, T3 BC546B, T4 BC546B, T5 BC546B, T6 BC546B

Commit message: Updated Schematics & Readme
Parts:
- added INT_TRG_CON: (no value), pinhead:PINHD-1X3
Connections:
- net BD1_TRIGGER: now also INT_TRG_CON.1
- net BD2_TRIGGER: now also INT_TRG_CON.2
- net SD_TRIGGER: now also INT_TRG_CON.3
Changed lines of the file:
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@@
 <part name="GND16" library="supply1" library_urn="urn:adsk.eagle:library:371" deviceset="GND" device=""/>
 <part name="P-1" library="supply1" deviceset="-12V" device=""/>
+<part name="INT_TRG_CON" library="pinhead" library_urn="urn:adsk.eagle:library:325" deviceset="PINHD-1X3" device="" package3d_urn="urn:adsk.eagle:package:22458/2"/>
 </parts>
 <sheets>
@@
 <instance part="P-1" gate="1" x="294.64" y="48.26" smashed="yes">
 <attribute name="VALUE" x="292.1" y="45.72" size="1.778" layer="96" rot="R90"/>
+</instance>
+<instance part="INT_TRG_CON" gate="A" x="256.54" y="284.48" smashed="yes">
+<attribute name="NAME" x="250.19" y="290.195" size="1.778" layer="95"/>
+<attribute name="VALUE" x="250.19" y="276.86" size="1.778" layer="96"/>
 </instance>
 </instances>
@@
 <wire x1="124.46" y1="147.32" x2="116.84" y2="147.32" width="0.1524" layer="91"/>
 <label x="116.84" y="147.32" size="1.778" layer="95" rot="R180" xref="yes"/>
+</segment>
+<segment>
+<pinref part="INT_TRG_CON" gate="A" pin="3"/>
+<wire x1="254" y1="281.94" x2="246.38" y2="281.94" width="0.1524" layer="91"/>
+<label x="246.38" y="281.94" size="1.778" layer="95" rot="R180" xref="yes"/>
 </segment>
 </net>
@@
 <label x="76.2" y="294.64" size="1.778" layer="95" rot="R180" xref="yes"/>
 </segment>
+<segment>
+<pinref part="INT_TRG_CON" gate="A" pin="1"/>
+<wire x1="254" y1="287.02" x2="241.3" y2="287.02" width="0.1524" layer="91"/>
+<label x="246.38" y="287.02" size="1.778" layer="95" rot="R180" xref="yes"/>
+</segment>
 </net>
 <net name="BD2_TRIGGER" class="0">
@@
 <pinref part="BD2_CON" gate="A" pin="1"/>
 </segment>
-</net>
+<segment>
+<pinref part="INT_TRG_CON" gate="A" pin="2"/>
+<wire x1="254" y1="284.48" x2="223.52" y2="284.48" width="0.1524" layer="91"/>
+<label x="223.52" y="284.48" size="1.778" layer="95" rot="R180" xref="yes"/>
+</segment>
+</net>

Commit message: Updated Schematics, Fixed Power Socket orientation
Parts:
- removed C11, C12: 10uf, resistor:CPOL-USE2.5-5
- added C16, C17: 10uf, resistor:CPOL-USE2.5-5
- C1, C10, C19, C35: value 47u/16v -> 47uF/16v
- C13, C2, C23: value 0.47u/50v -> .47uF/50v
- C14, C15, C25: value 0.056u -> .056uF
- C18: value 33u -> 33uF
- C20, C21: value 0.027u -> .027uF
- C22: value 0.0033u -> .0033uF
- C24: value 4.7u/50v -> 4.7uF/50v
- C26: value 0.0022u -> .0022uF
- C27: value 0.047 -> .047uF
- C28: value 0.0015u -> .0015uF
- C29, C30: value 0.0018u -> .0018uF
- C3, C4: value 0.056uf -> .056uF
- C31: value 0.01u -> .01uF
- C32, C34, C7, C8: value 1u/50v -> 1uF/50v
- C33: value 22p -> 22pF
- C5, C6: value 0.015uf -> .015uF
- C9: value 0.01uf -> .01uF
- D1, D2: value 1N4148DO35-7 -> 1N4148
- R17: device rcl:R-EU_0207/7 -> rcl:R-US_0207/7
Connections:
- net +12V: now also C17.+, PWR.10, PWR.9; no longer C12.+, PWR.1, PWR.2
- net -12V: now also C16.-, PWR.1, PWR.2; no longer C11.-, PWR.10, PWR.9
- net GND: now also C16.+, C17.-; no longer C11.+, C12.-
Other:
- moved on the sheet: C20, C24, C25, C28, C3, C4, C5, C6, D1, D2, PWR, R11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

Commit message: Fixed orentation SD Decay pot
Parts:
- R18: value 6.6k -> 3.3k
Changed lines of the file:
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@@
 <part name="C14" library="resistor" deviceset="C-EU" device="050-024X044" value=".056uF"/>
 <part name="C15" library="resistor" deviceset="C-EU" device="050-024X044" value=".056uF"/>
-<part name="R18" library="rcl" library_urn="urn:adsk.eagle:library:334" deviceset="R-US_" device="0207/7" package3d_urn="urn:adsk.eagle:package:23493/2" value="6.6k"/>
+<part name="R18" library="rcl" library_urn="urn:adsk.eagle:library:334" deviceset="R-US_" device="0207/7" package3d_urn="urn:adsk.eagle:package:23493/2" value="3.3k"/>
 <part name="R19" library="rcl" library_urn="urn:adsk.eagle:library:334" deviceset="R-US_" device="0207/7" package3d_urn="urn:adsk.eagle:package:23493/2" value="680k"/>
 <part name="GND11" library="supply1" deviceset="GND" device=""/>
